File: peak-read-amp/peak-read-amp.kicad_sch (KiCad schematic)
At the start: 44 parts, among them J1 Conn_01x02_Pin, J2 Conn_01x04_Pin, J3 Conn_01x04_Pin, U1 LM7808_TO220, U2 LM324, U3 LM324

Commit message: PCB version 1.0.1 to add mounting holes and clean up a few minor inconsistencies.  Upgraded to Kicad v9.
Changed lines of the file:
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@@
 (kicad_sch
-	(version 20231120)
+	(version 20250114)
 	(generator "eeschema")
-	(generator_version "8.0")
+	(generator_version "9.0")
 	(paper "A4")
 	(junction
@@
 		)
 	)
+	(embedded_fonts no)
 )
